Commit message: Fix : joint axes

File: ip010_gazebo/urdf/ip010.urdf.xacro (robot description, xacro)
@@ -1,4 +1,6 @@
 <?xml version="1.0" ?>
 <robot name="ip010" xmlns:xacro="http://www.ros.org/wiki/xacro">
+  <xacro:include filename="$(find ip010_description)/urdf/ip010.gazebo" />
+  <link name='base_footprint' />
   <link name="base_link">
     <inertial>
@@ -10,5 +12,5 @@
       <origin xyz="0 0 0" rpy="0 0 0" />
       <geometry>
-        <mesh filename="package://ip010_description/meshes/base_link.STL" />
+        <mesh filename="$(find ip010_description)/meshes/base_link.STL" />
       </geometry>
       <material name="">
@@ -19,8 +21,13 @@
       <origin xyz="0 0 0" rpy="0 0 0" />
       <geometry>
-        <mesh filename="package://ip010_description/meshes/base_link.STL" />
+        <mesh filename="$(find ip010_description)/meshes/base_link.STL" />
       </geometry>
     </collision>
   </link>
+  <joint name='base_link_joint' type='fixed'>
+    <origin rpy="0 0 0" xyz="0 0 0" />
+    <parent link="base_footprint" />
+    <child link="base_link" />
+  </joint>
   <link name="l_rear_wheel">
     <inertial>
@@ -32,5 +39,5 @@
       <origin xyz="0 0 0" rpy="0 0 0" />
       <geometry>
-        <mesh filename="package://ip010_description/meshes/l_rear_wheel.STL" />
+        <mesh filename="$(find ip010_description)/meshes/l_rear_wheel.STL" />
       </geometry>
       <material name="">
@@ -41,5 +48,5 @@
       <origin xyz="0 0 0" rpy="0 0 0" />
       <geometry>
-        <mesh filename="package://ip010_description/meshes/l_rear_wheel.STL" />
+        <mesh filename="$(find ip010_description)/meshes/l_rear_wheel.STL" />
       </geometry>
     </collision>
@@ -60,5 +67,5 @@
       <origin xyz="0 0 0" rpy="0 0 0" />
       <geometry>
-        <mesh filename="package://ip010_description/meshes/r_rear_wheel.STL" />
+        <mesh filename="$(find ip010_description)/meshes/r_rear_wheel.STL" />
       </geometry>
       <material name="">
@@ -69,5 +76,5 @@
       <origin xyz="0 0 0" rpy="0 0 0" />
       <geometry>
-        <mesh filename="package://ip010_description/meshes/r_rear_wheel.STL" />
+        <mesh filename="$(find ip010_description)/meshes/r_rear_wheel.STL" />
       </geometry>
     </collision>
@@ -88,5 +95,5 @@
       <origin xyz="0 0 0" rpy="0 0 0" />
       <geometry>
-        <mesh filename="package://ip010_description/meshes/center_lidar.STL" />
+        <mesh filename="$(find ip010_description)/meshes/center_lidar.STL" />
       </geometry>
       <material name="">
@@ -97,5 +104,5 @@
       <origin xyz="0 0 0" rpy="0 0 0" />
       <geometry>
-        <mesh filename="package://ip010_description/meshes/center_lidar.STL" />
+        <mesh filename="$(find ip010_description)/meshes/center_lidar.STL" />
       </geometry>
     </collision>
@@ -116,5 +123,5 @@
       <origin xyz="0 0 0" rpy="0 0 0" />
       <geometry>
-        <mesh filename="package://ip010_description/meshes/front_camera.STL" />
+        <mesh filename="$(find ip010_description)/meshes/front_camera.STL" />
       </geometry>
       <material name="">
@@ -125,5 +132,5 @@
       <origin xyz="0 0 0" rpy="0 0 0" />
       <geometry>
-        <mesh filename="package://ip010_description/meshes/front_camera.STL" />
+        <mesh filename="$(find ip010_description)/meshes/front_camera.STL" />
       </geometry>
     </collision>
