Commit message: Folder reordered

File: ip010_gazebo/urdf/ip010_description.urdf (robot description, URDF)
Before this commit: robot ip010, 7 links, 6 joints
Links:
- link base_link: geometry collision mesh filename=/home/kimsooyoung/ros2_ws/install/ip010_description/share/i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; visual mesh filename=/home/kimsooyoung/ros2_ws/install/ip010_description/share/i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
- link center_lidar: geometry collision mesh filename=/home/kimsooyoung/ros2_ws/install/ip010_description/share/i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; visual mesh filename=/home/kimsooyoung/ros2_ws/install/ip010_description/share/i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
- link front_ballcaster: geometry collision mesh filename=/home/kimsooyoung/ros2_ws/install/ip010_description/share/i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; visual mesh filename=/home/kimsooyoung/ros2_ws/install/ip010_description/share/i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
- link front_camera: geometry collision mesh filename=/home/kimsooyoung/ros2_ws/install/ip010_description/share/i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; visual mesh filename=/home/kimsooyoung/ros2_ws/install/ip010_description/share/i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
- link l_rear_wheel: geometry collision mesh filename=/home/kimsooyoung/ros2_ws/install/ip010_description/share/i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; visual mesh filename=/home/kimsooyoung/ros2_ws/install/ip010_description/share/i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
- link r_rear_wheel: geometry collision mesh filename=/home/kimsooyoung/ros2_ws/install/ip010_description/share/i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; visual mesh filename=/home/kimsooyoung/ros2_ws/install/ip010_description/share/i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

File: ip010_gazebo/urdf/ip010_description.urdf.xacro (robot description, xacro)
@@ -1,4 +1,6 @@
 <?xml version="1.0"?>
 <robot name="ip010" xmlns:xacro="http://www.ros.org/wiki/xacro">
+  <xacro:include filename="$(find ip010_gazebo)/urdf/ip010.gazebo" />
+  <link name='base_footprint' />
   <link name="base_link">
     <inertial>
@@ -10,5 +12,5 @@
       <origin xyz="0 0 0" rpy="0 0 0" />
       <geometry>
-        <mesh filename="package://ip010_description/meshes/new/base_link.STL" />
+        <mesh filename="$(find ip010_description)/meshes/base_link.STL" />
       </geometry>
       <material name="">
@@ -19,8 +21,13 @@
       <origin xyz="0 0 0" rpy="0 0 0" />
       <geometry>
-        <mesh filename="package://ip010_description/meshes/new/base_link.STL" />
+        <mesh filename="$(find ip010_description)/meshes/base_link.STL" />
       </geometry>
     </collision>
   </link>
+  <joint name='base_link_joint' type='fixed'>
+    <origin rpy="0 0 0" xyz="0 0 0" />
+    <parent link="base_footprint" />
+    <child link="base_link" />
+  </joint>
   <link name="l_rear_wheel">
     <inertial>
@@ -32,5 +39,5 @@
       <origin xyz="0 0 0" rpy="0 0 0" />
       <geometry>
-        <mesh filename="package://ip010_description/meshes/new/l_rear_wheel.STL" />
+        <mesh filename="$(find ip010_description)/meshes/l_rear_wheel.STL" />
       </geometry>
       <material name="">
@@ -41,9 +48,9 @@
       <origin xyz="0 0 0" rpy="0 0 0" />
       <geometry>
-        <mesh filename="package://ip010_description/meshes/new/l_rear_wheel.STL" />
+        <mesh filename="$(find ip010_description)/meshes/l_rear_wheel.STL" />
       </geometry>
     </collision>
   </link>
-  <joint name="l_rear_wheel" type="continuous">
+  <joint name="l_rear_wheel_joint" type="continuous">
     <origin xyz="-0.0945002035940863 0.11 0.0350003475684688" rpy="0 0 0" />
     <parent link="base_link" />
@@ -60,5 +67,5 @@
       <origin xyz="0 0 0" rpy="0 0 0" />
       <geometry>
-        <mesh filename="package://ip010_description/meshes/new/r_rear_wheel.STL" />
+        <mesh filename="$(find ip010_description)/meshes/r_rear_wheel.STL" />
       </geometry>
       <material name="">
@@ -69,9 +76,9 @@
       <origin xyz="0 0 0" rpy="0 0 0" />
       <geometry>
-        <mesh filename="package://ip010_description/meshes/new/r_rear_wheel.STL" />
+        <mesh filename="$(find ip010_description)/meshes/r_rear_wheel.STL" />
       </geometry>
     </collision>
   </link>
-  <joint name="r_rear_wheel" type="continuous">
+  <joint name="r_rear_wheel_joint" type="continuous">
     <origin xyz="-0.0944995996831282 -0.11 0.0350000447264209" rpy="0 0 0" />
     <parent link="base_link" />
@@ -88,5 +95,5 @@
       <origin xyz="0 0 0" rpy="0 0 0" />
       <geometry>
-        <mesh filename="package://ip010_description/meshes/new/front_ballcaster.STL" />
+        <mesh filename="$(find ip010_description)/meshes/front_ballcaster.STL" />
       </geometry>
       <material name="">
@@ -97,12 +104,13 @@
       <origin xyz="0 0 0" rpy="0 0 0" />
       <geometry>
-        <mesh filename="package://ip010_description/meshes/new/front_ballcaster.STL" />
+        <mesh filename="$(find ip010_description)/meshes/front_ballcaster.STL" />
       </geometry>
     </collision>
   </link>
-  <joint name="front_ballcaster" type="fixed">
+  <joint name="front_ballcaster_joint" type="fixed">
     <origin xyz="0.0879999994802632 0 0.000999753890741178" rpy="0 0 0" />
     <parent link="base_link" />
     <child link="front_ballcaster" />
+    <!-- <axis xyz="0 0 -1" /> -->
   </joint>
   <link name="center_lidar">
@@ -115,5 +123,5 @@
       <origin xyz="0 0 0" rpy="0 0 0" />
       <geometry>
-        <mesh filename="package://ip010_description/meshes/new/center_lidar.STL" />
+        <mesh filename="$(find ip010_description)/meshes/center_lidar.STL" />
       </geometry>
       <material name="">
@@ -124,9 +132,9 @@
       <origin xyz="0 0 0" rpy="0 0 0" />
       <geometry>
-        <mesh filename="package://ip010_description/meshes/new/center_lidar.STL" />
+        <mesh filename="$(find ip010_description)/meshes/center_lidar.STL" />
       </geometry>
     </collision>
   </link>
-  <joint name="center_lidar" type="fixed">
+  <joint name="center_lidar_joint" type="fixed">
     <origin xyz="-0.0321033068699902 -4.99877536184437E-05 0.119000000000201" rpy="0 0 0" />
     <parent link="base_link" />
@@ -143,5 +151,5 @@
       <origin xyz="0 0 0" rpy="0 0 0" />
       <geometry>
-        <mesh filename="package://ip010_description/meshes/new/front_camera.STL" />
+        <mesh filename="$(find ip010_description)/meshes/front_camera.STL" />
       </geometry>
       <material name="">
@@ -152,9 +160,9 @@
       <origin xyz="0 0 0" rpy="0 0 0" />
       <geometry>
-        <mesh filename="package://ip010_description/meshes/new/front_camera.STL" />
+        <mesh filename="$(find ip010_description)/meshes/front_camera.STL" />
       </geometry>
     </collision>
   </link>
-  <joint name="front_camera" type="fixed">
+  <joint name="front_camera_joint" type="fixed">
     <origin xyz="0.141847512071907 -0.000215421199799998 0.0680000000002" rpy="0 0 0" />
     <parent link="base_link" />
